Commit message: Update det_racecar.xacro

File: det_racecar.xacro (robot description, xacro)
@@ -2,6 +2,6 @@
 <!-- A simple model of the racecar for rviz -->
 <robot xmlns:xacro="http://www.ros.org/wiki/xacro" name="$det_racecar">
-  <xacro:property name="wheelbase" value="0.3302" />
-  <xacro:property name="width" value="0.2032" />
+  <xacro:property name="wheelbase" value="0.5002" />
+  <xacro:property name="width" value="0.3632" />
   <xacro:property name="height" value="0.1" />
   <xacro:property name="ground_offset" value="0.04" />
